File: tt-ecp5-cb.kicad_sch (KiCad schematic)
At the start: 27 parts, among them J1 Conn_02x05_Odd_Even, J2 TT06_BREAKOUT_REVA, Q1 Q_NMOS_GSD, U1 LFE5U_25_CABGA256, U2 TLV62565DBVx, U3 TLV73325PDBV

Commit message: Silkscreen, test pads
Parts:
- added TP1, TP2, TP3, TP4, TP5: TestPoint, TestPoint:TestPoint_Pad_2.0x2.0mm, symbol Connector:TestPoint
Connections:
- net +1V1: now also TP4.1
- net +2V5: now also TP5.1
- net at R5.2, U1.P10 (CFG_1): now also TP2.1
- net at R4.2, U1.N10 (CFG_0): now also TP1.1
- net at R6.2, U1.R10 (CFG_2): now also TP3.1
Other:
- moved on the sheet: R4, R5, R6

Commit message: First version
Parts:
- C1, C4: footprint Capacitor_SMD:C_0603_1608Metric -> Capacitor_SMD:C_0402_1005Metric
Changed lines of the file:
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@@
 			)
 		)
-		(property "Footprint" "Capacitor_SMD:C_0603_1608Metric"
+		(property "Footprint" "Capacitor_SMD:C_0402_1005Metric"
 			(at 103.8352 53.34 0)
 			(effects
@@
 			)
 		)
-		(property "Footprint" "Capacitor_SMD:C_0603_1608Metric"
+		(property "Footprint" "Capacitor_SMD:C_0402_1005Metric"
 			(at 40.3352 57.15 0)
 			(effects
